File: pcb/feb42.kicad_sch (KiCad schematic)
At the start: 343 parts, among them J1 Conn_01x04_Socket, Q1 2N7002, Q2 2N7002, U1 STM32F411CEU6

Commit message: rev2
Parts:
- BRD2: LCSC (none) -> C2128
- D1: LCSC (none) -> C7371898
- LM1: LCSC (none) -> C82045
- Q1, Q2: LCSC (none) -> C8545
- R2: value 5.1k -> 1.5k; LCSC (none) -> C25867
- R4, R5, R8: LCSC (none) -> C25744
- R6: LCSC (none) -> C25076
- R7: LCSC (none) -> C11702
- R9: LCSC (none) -> C25741
- U1: LCSC (none) -> C60420
Changed lines of the file:
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@@
 			)
 		)
+		(property "LCSC" "C2128"
+			(at 49.53 72.39 0)
+			(effects
+				(font
+					(size 1.27 1.27)
+				)
+				(hide yes)
+			)
+		)
 		(pin "1"
 		)
@@
 			)
 		)
+		(property "LCSC" "C11702"
+			(at 45.72 39.37 90)
+			(effects
+				(font
+					(size 1.27 1.27)
+				)
+				(hide yes)
+			)
+		)
 		(pin "1"
 		)
@@
 			)
 		)
+		(property "LCSC" "C8545"
+			(at 60.96 39.37 0)
+			(effects
+				(font
+					(size 1.27 1.27)
+				)
+				(hide yes)
+			)
+		)
 		(pin "2"
 		)
@@
 			)
 		)
+		(property "LCSC" "C8545"
+			(at 82.55 59.69 0)
+			(effects
+				(font
+					(size 1.27 1.27)
+				)
+				(hide yes)
+			)
+		)
 		(pin "2"
 		)
@@
 			)
 		)
+		(property "LCSC" "C60420"
+			(at 165.1 88.9 0)
+			(effects
+				(font
+					(size 1.27 1.27)
+				)
+				(hide yes)
+			)
+		)
 		(pin "27"
 		)
@@
 			)
 		)
+		(property "LCSC" "C25076"
+			(at 73.66 44.45 90)
+			(effects
+				(font
+					(size 1.27 1.27)
+				)
+				(hide yes)
+			)
+		)
 		(pin "1"
 		)
@@
 			)
 		)
-		(property "LCSC" ""
+		(property "LCSC" "C25741"
 			(at 74.93 55.88 90)
 			(effects
@@
 			)
 		)
+		(property "LCSC" "C25744"
+			(at 85.09 68.58 90)
+			(effects
+				(font
+					(size 1.27 1.27)
+				)
+				(hide yes)
+			)
+		)
 		(pin "1"
 		)
@@
 			)
 		)
+		(property "LCSC" "C7371898"
+			(at 200.66 62.23 90)
+			(effects
+				(font
+					(size 1.27 1.27)
+				)
+				(hide yes)
+			)
+		)
 		(pin "1"
 		)
@@
 			)
 		)
-		(property "Value" "5.1k"
+		(property "Value" "1.5k"
 			(at 206.502 57.15 90)
 			(effects
@@
 			)
 		)
+		(property "LCSC" "C25867"
+			(at 204.47 57.15 90)
+			(effects
+				(font
+					(size 1.27 1.27)
+				)
+				(hide yes)
+			)
+		)
 		(pin "1"
 		)
@@
 			)
 		)
+		(property "LCSC" "C25744"
+			(at 68.58 59.69 90)
+			(effects
+				(font
+					(size 1.27 1.27)
+				)
+				(hide yes)
+			)
+		)
 		(pin "1"
 		)
@@
 			)
 		)
+		(property "LCSC" "C25744"
+			(at 53.34 35.56 90)
+			(effects
+				(font
+					(size 1.27 1.27)
+				)
+				(hide yes)
+			)
+		)
 		(pin "1"
 		)
@@
 			(effects
 				(font
+					(size 1.27 1.27)
+				)
+				(hide yes)
+			)
+		)
+		(property "LCSC" "C82045"
+			(at 380.365 415.29 90)
+			(effects
+				(font
